File: KiCad/NanoFox80/NanoFox80.kicad_sch (KiCad schematic)
At the start: 58 parts, among them J101 Conn_01x02, J102 Conn_01x02, J103 Conn_01x02, J104 Conn_01x02, J111 DB9 Female, J112 Conn_01x02, J113 Conn_01x02, J115 Conn_01x02, P101 ISP/PDI, Q101 BSS84W-7-F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

Commit message: Update NanoFox80.kicad_sch
Schematic tweaks.
Parts:
- C106: value 15-60pF -> (none)
- C118: value TBD pF -> (none)
- D102: value 4.7V -> (none)
- Q103: value DTC113Z -> (none); Digi-Key Part No. (none) -> 264-RN1426TE85LFCT-ND; Link (none) -> https://www.digikey.com/en/products/detail/toshiba-semicond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; Manufacturer (none) -> Toshiba Semiconductor and Storage
- R103: value 10 -> (none)
Changed lines of the file:
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@@
       (effects (font (size 1.27 1.27)) (justify right))
     )
-    (property "Value" "15-60pF" (id 1) (at 201.7014 57.7092 0)
+    (property "Value" "" (id 1) (at 201.7014 57.7092 0)
       (effects (font (size 1.27 1.27)) (justify right))
     )
@@
       (effects (font (size 1.27 1.27)) (justify left))
     )
-    (property "Value" "DTC113Z" (id 1) (at 186.182 38.5322 0)
+    (property "Value" "" (id 1) (at 186.182 38.5322 0)
       (effects (font (size 1.27 1.27)) (justify left))
     )
@@
     (property "Datasheet" "" (id 3) (at 181.61 36.83 0)
       (effects (font (size 1.27 1.27)) (justify left) hide)
+    )
+    (property "Digi-Key Part No." "264-RN1426TE85LFCT-ND" (id 4) (at 181.61 36.83 0)
+      (effects (font (size 1.27 1.27)) hide)
+    )
+    (property "Link" "https://www.digikey.com/en/products/detail/toshiba-semiconductor-and-storage/RN1426TE85LF/2330276" (id 5) (at 181.61 36.83 0)
+      (effects (font (size 1.27 1.27)) hide)
+    )
+    (property "Manufacturer" "Toshiba Semiconductor and Storage" (id 6) (at 181.61 36.83 0)
+      (effects (font (size 1.27 1.27)) hide)
     )
     (pin "1")
@@
       (effects (font (size 1.27 1.27)) (justify left))
     )
-    (property "Value" "4.7V" (id 1) (at 185.928 55.0422 90)
+    (property "Value" "" (id 1) (at 185.928 55.0422 90)
       (effects (font (size 1.27 1.27)) (justify left))
     )
@@
     (in_bom yes) (on_board yes) (fields_autoplaced)
     (property "Reference" "R103" (id 0) (at 191.77 44.9412 90))
-    (property "Value" "10" (id 1) (at 191.77 47.4781 90))
+    (property "Value" "" (id 1) (at 191.77 47.4781 90))
     (property "Footprint" "" (id 2) (at 191.77 49.53 0)
       (effects (font (size 1.27 1.27)) hide)
@@
       (effects (font (size 1.27 1.27)) (justify left))
     )
-    (property "Value" "TBD pF" (id 1) (at 213.36 58.42 0)
+    (property "Value" "" (id 1) (at 213.36 58.42 0)
       (effects (font (size 1.27 1.27)) (justify left))
     )
@@
     )
     (path "/0e1e7a3c-c50c-4d42-9572-0d002900c69d"
-      (reference "C106") (unit 1) (value "15-60pF") (footprint "Capacitor_THT:CP_Radial_Ceramic_Trimmer_D9.4mm_P8.00mm")
+      (reference "C106") (unit 1) (value "NP") (footprint "Capacitor_THT:CP_Radial_Ceramic_Trimmer_D9.4mm_P8.00mm")
     )
     (path "/1230aad1-fe96-4be0-9f04-1e46bf447e94"
@@
     )
     (path "/e185d3e9-1152-453e-9913-3041132c8b39"
-      (reference "C118") (unit 1) (value "TBD pF") (footprint "Capacitor_SMD:C_0805_2012Metric")
+      (reference "C118") (unit 1) (value "NP") (footprint "Capacitor_SMD:C_0805_2012Metric")
     )
     (path "/46155e87-3819-47f9-b3a7-1d0e71924957"
@@
     )
     (path "/9a362b03-69ee-4b1f-b653-32a8ac132ea9"
-      (reference "D102") (unit 1) (value "4.7V") (footprint "")
+      (reference "D102") (unit 1) (value "NP") (footprint "")
     )
     (path "/494208f9-e0ca-4027-9207-cba02c8b4cf6"
@@
     )
     (path "/7e4f8b88-6c4b-4ba5-bc05-ae0251584d83"
-      (reference "Q103") (unit 1) (value "DTC113Z") (footprint "")
+      (reference "Q103") (unit 1) (value "RN1426TE85LF") (footprint "Package_TO_SOT_SMD:SC-59")
     )
     (path "/68b55295-fe67-43f3-942f-ec08960df788"
@@
     )
     (path "/bec9562c-6b4c-48ba-b645-29b85449b6e2"
-      (reference "R103") (unit 1) (value "10") (footprint "")
+      (reference "R103") (unit 1) (value "10") (footprint "Resistor_SMD:R_0805_2012Metric")
     )
     (path "/c4a0b625-0796-4f97-b5bb-d859e812789a"

Commit message: Update NanoFox80.kicad_sch
More tweaks
Connections:
- net Antenna: now also AE101.2 (A), C102.1, J102.2 (Pin_2); no longer C105.1, C115.1, L101.1, L102.1
- new net: C105.1, C115.1, L101.1, L102.1
Other:
- moved on the sheet: C102, C119, L102
Changed lines of the file:
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@@
   (junction (at 107.95 151.13) (diameter 0) (color 0 0 0 0)
   )
-  (junction (at 260.35 49.53) (diameter 0) (color 0 0 0 0)
+  (junction (at 254 49.53) (diameter 0) (color 0 0 0 0)
   )
   (junction (at 137.16 55.88) (diameter 0) (color 0 0 0 0)
@@
   (junction (at 80.01 165.1) (diameter 0) (color 0 0 0 0)
   )
+  (junction (at 262.89 49.53) (diameter 0) (color 0 0 0 0)
+  )
   (junction (at 80.01 151.13) (diameter 0) (color 0 0 0 0)
   )
@@
   )
   (junction (at 62.23 63.5) (diameter 0) (color 0 0 0 0)
-  )
-  (junction (at 238.76 49.53) (diameter 0) (color 0 0 0 0)
   )
   (junction (at 134.62 101.6) (diameter 0) (color 0 0 0 0)
@@
     (stroke (width 0) (type default) (color 0 0 0 0))
   )
-  (wire (pts (xy 238.76 49.53) (xy 243.84 49.53))
+  (wire (pts (xy 236.22 49.53) (xy 238.76 49.53))
     (stroke (width 0) (type default) (color 0 0 0 0))
   )
@@
     (stroke (width 0) (type default) (color 0 0 0 0))
   )
+  (wire (pts (xy 262.89 45.72) (xy 262.89 49.53))
+    (stroke (width 0) (type default) (color 0 0 0 0))
+  )
   (wire (pts (xy 80.01 165.1) (xy 80.01 162.56))
     (stroke (width 0) (type default) (color 0 0 0 0))
@@
     (stroke (width 0) (type default) (color 0 0 0 0))
   )
+  (wire (pts (xy 262.89 49.53) (xy 267.97 49.53))
+    (stroke (width 0) (type default) (color 0 0 0 0))
+  )
   (wire (pts (xy 41.91 151.13) (xy 73.66 151.13))
     (stroke (width 0) (type default) (color 0 0 0 0))
@@
     (stroke (width 0) (type default) (color 0 0 0 0))
   )
-  (wire (pts (xy 238.76 43.18) (xy 241.3 43.18))
-    (stroke (width 0) (type default) (color 0 0 0 0))
-  )
-  (wire (pts (xy 236.22 49.53) (xy 238.76 49.53))
-    (stroke (width 0) (type default) (color 0 0 0 0))
-  )
-  (wire (pts (xy 266.7 49.53) (xy 267.97 49.53))
+  (wire (pts (xy 260.35 49.53) (xy 262.89 49.53))
     (stroke (width 0) (type default) (color 0 0 0 0))
   )
@@
     (stroke (width 0) (type default) (color 0 0 0 0))
   )
-  (wire (pts (xy 256.54 49.53) (xy 260.35 49.53))
+  (wire (pts (xy 251.46 49.53) (xy 254 49.53))
     (stroke (width 0) (type default) (color 0 0 0 0))
   )
@@
     (stroke (width 0) (type default) (color 0 0 0 0))
   )
-  (wire (pts (xy 260.35 49.53) (xy 260.35 53.34))
+  (wire (pts (xy 254 49.53) (xy 254 53.34))
     (stroke (width 0) (type default) (color 0 0 0 0))
   )
@@
     (stroke (width 0) (type default) (color 0 0 0 0))
   )
-  (wire (pts (xy 260.35 49.53) (xy 261.62 49.53))
+  (wire (pts (xy 254 49.53) (xy 255.27 49.53))
     (stroke (width 0) (type default) (color 0 0 0 0))
   )
@@
   )
   (wire (pts (xy 62.23 63.5) (xy 62.23 66.04))
-    (stroke (width 0) (type default) (color 0 0 0 0))
-  )
-  (wire (pts (xy 238.76 49.53) (xy 238.76 43.18))
     (stroke (width 0) (type default) (color 0 0 0 0))
   )
@@
     )
   )
-  (global_label "Antenna" (shape output) (at 241.3 43.18 0) (fields_autoplaced)
+  (global_label "Antenna" (shape output) (at 262.89 45.72 90) (fields_autoplaced)
     (effects (font (size 1 1)) (justify left))
-    (property "Intersheet References" "${INTERSHEET_REFS}" (id 0) (at 249.1048 43.1175 0)
+    (property "Intersheet References" "${INTERSHEET_REFS}" (id 0) (at 262.8275 37.9152 90)
       (effects (font (size 1 1)) (justify left) hide)
     )
@@
     (pin "1")
   )
-  (symbol (lib_id "pspice:INDUCTOR") (at 250.19 49.53 0) (unit 1)
-    (in_bom yes) (on_board yes) (fields_autoplaced)
-    (property "Reference" "L102" (id 0) (at 250.19 44.6872 0))
-    (property "Value" "TBD nF" (id 1) (at 250.19 47.2241 0))
-    (property "Footprint" "" (id 2) (at 250.19 49.53 0)
-      (effects (font (size 1.27 1.27)) hide)
-    )
-    (property "Datasheet" "~" (id 3) (at 250.19 49.53 0)
+  (symbol (lib_id "pspice:INDUCTOR") (at 245.11 49.53 0) (unit 1)
+    (in_bom yes) (on_board yes) (fields_autoplaced)
+    (property "Reference" "L102" (id 0) (at 245.11 44.6872 0))
+    (property "Value" "TBD nF" (id 1) (at 245.11 47.2241 0))
+    (property "Footprint" "" (id 2) (at 245.11 49.53 0)
+      (effects (font (size 1.27 1.27)) hide)
+    )
+    (property "Datasheet" "~" (id 3) (at 245.11 49.53 0)
       (effects (font (size 1.27 1.27)) hide)
     )
@@
     (pin "1")
   )
-  (symbol (lib_id "Device:C_Small") (at 260.35 55.88 0) (unit 1)
-    (in_bom yes) (on_board yes)
-    (property "Reference" "C119" (id 0) (at 254 53.34 0)
+  (symbol (lib_id "Device:C_Small") (at 254 55.88 0) (unit 1)
+    (in_bom yes) (on_board yes)
+    (property "Reference" "C119" (id 0) (at 247.65 53.34 0)
       (effects (font (size 1.27 1.27)) (justify left))
     )
-    (property "Value" "TBD pF" (id 1) (at 252.73 58.42 0)
+    (property "Value" "TBD pF" (id 1) (at 246.38 58.42 0)
       (effects (font (size 1.27 1.27)) (justify left))
     )
-    (property "Footprint" "Capacitor_SMD:C_0805_2012Metric" (id 2) (at 260.35 55.88 0)
-      (effects (font (size 1.27 1.27)) hide)
-    )
-    (property "Datasheet" "~" (id 3) (at 260.35 55.88 0)
-      (effects (font (size 1.27 1.27)) hide)
-    )
-    (property "Digi-Key Part No." "478-1274-1-ND" (id 4) (at 260.35 55.88 0)
-      (effects (font (size 1.27 1.27)) hide)
-    )
-    (property "Manufacturer" "KYOCERA AVX" (id 5) (at 260.35 55.88 0)
-      (effects (font (size 1.27 1.27)) hide)
-    )
-    (property "Manufacturer PN" "08052A221JAT2A" (id 6) (at 260.35 55.88 0)
-      (effects (font (size 1.27 1.27)) hide)
-    )
-    (property "Description" "CAP CER 220PF 200V C0G/NP0 0805" (id 7) (at 260.35 55.88 0)
+    (property "Footprint" "Capacitor_SMD:C_0805_2012Metric" (id 2) (at 254 55.88 0)
+      (effects (font (size 1.27 1.27)) hide)
+    )
+    (property "Datasheet" "~" (id 3) (at 254 55.88 0)
+      (effects (font (size 1.27 1.27)) hide)
+    )
+    (property "Digi-Key Part No." "478-1274-1-ND" (id 4) (at 254 55.88 0)
+      (effects (font (size 1.27 1.27)) hide)
+    )
+    (property "Manufacturer" "KYOCERA AVX" (id 5) (at 254 55.88 0)
+      (effects (font (size 1.27 1.27)) hide)
+    )
+    (property "Manufacturer PN" "08052A221JAT2A" (id 6) (at 254 55.88 0)
+      (effects (font (size 1.27 1.27)) hide)
+    )
+    (property "Description" "CAP CER 220PF 200V C0G/NP0 0805" (id 7) (at 254 55.88 0)
       (effects (font (size 1.27 1.27)) hide)
     )
@@
     (pin "1")
   )
-  (symbol (lib_id "power:GND") (at 260.35 58.42 0) (unit 1)
-    (in_bom yes) (on_board yes) (fields_autoplaced)
-    (property "Reference" "#PWR0156" (id 0) (at 260.35 64.77 0)
-      (effects (font (size 1.27 1.27)) hide)
-    )
-    (property "Value" "GND" (id 1) (at 260.35 62.8634 0)
-      (effects (font (size 1.27 1.27)) hide)
-    )
-    (property "Footprint" "" (id 2) (at 260.35 58.42 0)
-      (effects (font (size 1.27 1.27)) hide)
-    )
-    (property "Datasheet" "" (id 3) (at 260.35 58.42 0)
+  (symbol (lib_id "power:GND") (at 254 58.42 0) (unit 1)
+    (in_bom yes) (on_board yes) (fields_autoplaced)
+    (property "Reference" "#PWR0156" (id 0) (at 254 64.77 0)
+      (effects (font (size 1.27 1.27)) hide)
+    )
+    (property "Value" "GND" (id 1) (at 254 62.8634 0)
+      (effects (font (size 1.27 1.27)) hide)
+    )
+    (property "Footprint" "" (id 2) (at 254 58.42 0)
+      (effects (font (size 1.27 1.27)) hide)
+    )
+    (property "Datasheet" "" (id 3) (at 254 58.42 0)
       (effects (font (size 1.27 1.27)) hide)
     )
@@
     (pin "1")
   )
-  (symbol (lib_id "Device:C_Small") (at 264.16 49.53 270) (unit 1)
-    (in_bom yes) (on_board yes)
-    (property "Reference" "C102" (id 0) (at 264.16 45.72 90))
-    (property "Value" "100nF" (id 1) (at 265.43 53.34 90))
-    (property "Footprint" "Capacitor_SMD:C_0805_2012Metric_Pad1.18x1.45mm_HandSolder" (id 2) (at 264.16 49.53 0)
-      (effects (font (size 1.27 1.27)) hide)
-    )
-    (property "Datasheet" "~" (id 3) (at 264.16 49.53 0)
-      (effects (font (size 1.27 1.27)) hide)
-    )
-    (property "Digi-Key Part No." "445-5203-1-ND" (id 4) (at 264.16 49.53 0)
-      (effects (font (size 1.27 1.27)) hide)
-    )
-    (property "Manufacturer" "TDK Corporation" (id 5) (at 264.16 49.53 0)
-      (effects (font (size 1.27 1.27)) hide)
-    )
-    (property "Manufacturer PN" "C2012X7S2A474K125AB" (id 6) (at 264.16 49.53 0)
-      (effects (font (size 1.27 1.27)) hide)
-    )
-    (property "Description" "CAP CER 0.47UF 100V X7S 0805" (id 7) (at 264.16 49.53 0)
-      (effects (font (size 1.27 1.27)) hide)
-    )
+  (symbol (lib_id "Device:C_Small") (at 257.81 49.53 270) (unit 1)
+    (in_bom yes) (on_board yes)
+    (property "Reference" "C102" (id 0) (at 257.81 45.72 90))
+    (property "Value" "100nF" (id 1) (at 259.08 53.34 90))
+    (property "Footprint" "Capacitor_SMD:C_0805_2012Metric_Pad1.18x1.45mm_HandSolder" (id 2) (at 257.81 49.53 0)
+      (effects (font (size 1.27 1.27)) hide)
+    )
+    (property "Datasheet" "~" (id 3) (at 257.81 49.53 0)
+      (effects (font (size 1.27 1.27)) hide)
+    )
+    (property "Digi-Key Part No." "445-5203-1-ND" (id 4) (at 257.81 49.53 0)
+      (effects (font (size 1.27 1.27)) hide)
+    )
+    (property "Manufacturer" "TDK Corporation" (id 5) (at 257.81 49.53 0)
+      (effects (font (size 1.27 1.27)) hide)
+    )
+    (property "Manufacturer PN" "C2012X7S2A474K125AB" (id 6) (at 257.81 49.53 0)
+      (effects (font (size 1.27 1.27)) hide)
+    )
+    (property "Description" "CAP CER 0.47UF 100V X7S 0805" (id 7) (at 257.81 49.53 0)
+      (effects (font (size 1.27 1.27)) hide)
+    )

Commit message: Update NanoFox80.kicad_sch
Schematic tweak - added cap across switch
Parts:
- added C?: 100nF, Capacitor_SMD:C_0805_2012Metric_Pad1.18x1.45mm_HandSolder, symbol Device:C_Small
- C106, C118, D102: value (none) -> NP
- Q103: value (none) -> RN1426TE85LF; footprint (none) -> Package_TO_SOT_SMD:SC-59
- R103: value (none) -> 10; footprint (none) -> Resistor_SMD:R_0805_2012Metric
Connections:
- net GND: now also C?.2
- net at D105.1 (K), J112.2 (Pin_2), Q101.1 (G)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: now also C?.1
Other:
- moved on the sheet: J112
Changed lines of the file:
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@@
   (junction (at 107.95 151.13) (diameter 0) (color 0 0 0 0)
   )
+  (junction (at 68.58 165.1) (diameter 0) (color 0 0 0 0)
+  )
   (junction (at 254 49.53) (diameter 0) (color 0 0 0 0)
   )
@@
   (junction (at 39.37 34.29) (diameter 0) (color 0 0 0 0)
   )
+  (junction (at 68.58 151.13) (diameter 0) (color 0 0 0 0)
+  )
   (junction (at 26.67 69.85) (diameter 0) (color 0 0 0 0)
   )
@@
   (junction (at 88.9 165.1) (diameter 0) (color 0 0 0 0)
   )
-  (junction (at 73.66 151.13) (diameter 0) (color 0 0 0 0)
+  (junction (at 63.5 151.13) (diameter 0) (color 0 0 0 0)
   )
   (junction (at 31.75 151.13) (diameter 0) (color 0 0 0 0)
@@
   (no_connect (at 148.59 130.81))
   (no_connect (at 148.59 140.97))
-  (wire (pts (xy 73.66 158.75) (xy 73.66 165.1))
+  (wire (pts (xy 63.5 158.75) (xy 63.5 165.1))
     (stroke (width 0) (type default) (color 0 0 0 0))
   )
@@
     (stroke (width 0) (type default) (color 0 0 0 0))
   )
-  (wire (pts (xy 73.66 165.1) (xy 80.01 165.1))
+  (wire (pts (xy 63.5 165.1) (xy 68.58 165.1))
     (stroke (width 0) (type default) (color 0 0 0 0))
   )
@@
     (stroke (width 0) (type default) (color 0 0 0 0))
   )
-  (wire (pts (xy 41.91 151.13) (xy 73.66 151.13))
+  (wire (pts (xy 41.91 151.13) (xy 63.5 151.13))
     (stroke (width 0) (type default) (color 0 0 0 0))
   )
@@
     (stroke (width 0) (type default) (color 0 0 0 0))
   )
+  (wire (pts (xy 68.58 165.1) (xy 80.01 165.1))
+    (stroke (width 0) (type default) (color 0 0 0 0))
+  )
   (wire (pts (xy 15.24 96.52) (xy 41.91 96.52))
     (stroke (width 0) (type default) (color 0 0 0 0))
@@
     (stroke (width 0) (type default) (color 0 0 0 0))
   )
-  (wire (pts (xy 73.66 156.21) (xy 73.66 151.13))
+  (wire (pts (xy 63.5 156.21) (xy 63.5 151.13))
     (stroke (width 0) (type default) (color 0 0 0 0))
   )
@@
     (stroke (width 0) (type default) (color 0 0 0 0))
   )
+  (wire (pts (xy 68.58 160.02) (xy 68.58 165.1))
+    (stroke (width 0) (type default) (color 0 0 0 0))
+  )
   (wire (pts (xy 139.7 88.9) (xy 139.7 101.6))
     (stroke (width 0) (type default) (color 0 0 0 0))
@@
     (stroke (width 0) (type default) (color 0 0 0 0))
   )
-  (wire (pts (xy 73.66 151.13) (xy 80.01 151.13))
+  (wire (pts (xy 63.5 151.13) (xy 68.58 151.13))
     (stroke (width 0) (type default) (color 0 0 0 0))
   )
@@
     (stroke (width 0) (type default) (color 0 0 0 0))
   )
+  (wire (pts (xy 68.58 151.13) (xy 68.58 154.94))
+    (stroke (width 0) (type default) (color 0 0 0 0))
+  )
   (wire (pts (xy 199.39 49.53) (xy 199.39 53.34))
     (stroke (width 0) (type default) (color 0 0 0 0))
@@
     (stroke (width 0) (type default) (color 0 0 0 0))
   )
+  (wire (pts (xy 68.58 151.13) (xy 80.01 151.13))
+    (stroke (width 0) (type default) (color 0 0 0 0))
+  )
   (wire (pts (xy 77.47 99.06) (xy 93.98 99.06))
     (stroke (width 0) (type default) (color 0 0 0 0))
@@
       (effects (font (size 1.27 1.27)) (justify right))
     )
-    (property "Value" "" (id 1) (at 201.7014 57.7092 0)
+    (property "Value" "NP" (id 1) (at 201.7014 57.7092 0)
       (effects (font (size 1.27 1.27)) (justify right))
     )
@@
     (pin "2")
   )
+  (symbol (lib_id "Device:C_Small") (at 68.58 157.48 0) (unit 1)
+    (in_bom yes) (on_board yes)
+    (property "Reference" "C?" (id 0) (at 64.77 157.48 90))
+    (property "Value" "100nF" (id 1) (at 72.39 156.21 90))
+    (property "Footprint" "Capacitor_SMD:C_0805_2012Metric_Pad1.18x1.45mm_HandSolder" (id 2) (at 68.58 157.48 0)
+      (effects (font (size 1.27 1.27)) hide)
+    )
+    (property "Datasheet" "~" (id 3) (at 68.58 157.48 0)
+      (effects (font (size 1.27 1.27)) hide)
+    )
+    (property "Digi-Key Part No." "445-5203-1-ND" (id 4) (at 68.58 157.48 0)
+      (effects (font (size 1.27 1.27)) hide)
+    )
+    (property "Manufacturer" "TDK Corporation" (id 5) (at 68.58 157.48 0)
+      (effects (font (size 1.27 1.27)) hide)
+    )
+    (property "Manufacturer PN" "C2012X7S2A474K125AB" (id 6) (at 68.58 157.48 0)
+      (effects (font (size 1.27 1.27)) hide)
+    )
+    (property "Description" "CAP CER 0.47UF 100V X7S 0805" (id 7) (at 68.58 157.48 0)
+      (effects (font (size 1.27 1.27)) hide)
+    )
+    (pin "1")
+    (pin "2")
+  )
   (symbol (lib_id "Regulator_Linear:LP2985-3.3") (at 49.53 36.83 0) (unit 1)
     (in_bom yes) (on_board yes)
@@
       (effects (font (size 1.27 1.27)) (justify left))
     )
-    (property "Value" "" (id 1) (at 186.182 38.5322 0)
+    (property "Value" "RN1426TE85LF" (id 1) (at 186.182 38.5322 0)
       (effects (font (size 1.27 1.27)) (justify left))
     )
-    (property "Footprint" "" (id 2) (at 181.61 36.83 0)
+    (property "Footprint" "Package_TO_SOT_SMD:SC-59" (id 2) (at 181.61 36.83 0)
       (effects (font (size 1.27 1.27)) (justify left) hide)
     )
@@
       (effects (font (size 1.27 1.27)) (justify left))
     )
-    (property "Value" "" (id 1) (at 185.928 55.0422 90)
+    (property "Value" "NP" (id 1) (at 185.928 55.0422 90)
       (effects (font (size 1.27 1.27)) (justify left))
     )
@@
       (effects (font (size 1.27 1.27)) hide)
     )
-    (property "Value" "" (id 1) (at 90.17 174.2242 0))
+    (property "Value" "+VSW" (id 1) (at 90.17 174.2242 0))
     (property "Footprint" "" (id 2) (at 90.17 177.8 0)
       (effects (font (size 1.27 1.27)) hide)
@@
     (in_bom yes) (on_board yes) (fields_autoplaced)
     (property "Reference" "R103" (id 0) (at 191.77 44.9412 90))
-    (property "Value" "" (id 1) (at 191.77 47.4781 90))
-    (property "Footprint" "" (id 2) (at 191.77 49.53 0)
+    (property "Value" "10" (id 1) (at 191.77 47.4781 90))
+    (property "Footprint" "Resistor_SMD:R_0805_2012Metric" (id 2) (at 191.77 49.53 0)
       (effects (font (size 1.27 1.27)) hide)
     )
@@
     (pin "4")
   )
-  (symbol (lib_id "Connector_Generic:Conn_01x02") (at 68.58 158.75 180) (unit 1)
+  (symbol (lib_id "Connector_Generic:Conn_01x02") (at 58.42 158.75 180) (unit 1)
     (in_bom yes) (on_board yes)
-    (property "Reference" "J112" (id 0) (at 66.04 158.75 90))
-    (property "Value" "Conn_01x02" (id 1) (at 68.58 161.1829 0)
+    (property "Reference" "J112" (id 0) (at 55.88 158.75 90))
+    (property "Value" "Conn_01x02" (id 1) (at 58.42 161.1829 0)
       (effects (font (size 1.27 1.27)) hide)
     )
-    (property "Footprint" "Connector_PinSocket_2.54mm:PinSocket_1x02_P2.54mm_Vertical" (id 2) (at 68.58 158.75 0)
+    (property "Footprint" "Connector_PinSocket_2.54mm:PinSocket_1x02_P2.54mm_Vertical" (id 2) (at 58.42 158.75 0)
       (effects (font (size 1.27 1.27)) hide)
     )
-    (property "Datasheet" "~" (id 3) (at 68.58 158.75 0)
+    (property "Datasheet" "~" (id 3) (at 58.42 158.75 0)
       (effects (font (size 1.27 1.27)) hide)
     )
@@
       (effects (font (size 1.27 1.27)) (justify left))
     )
-    (property "Value" "" (id 1) (at 213.36 58.42 0)
+    (property "Value" "NP" (id 1) (at 213.36 58.42 0)
       (effects (font (size 1.27 1.27)) (justify left))
     )
@@
       (reference "C203") (unit 1) (value "100nF") (footprint "Capacitor_SMD:C_0805_2012Metric_Pad1.18x1.45mm_HandSolder")
     )
+    (path "/6ff25e28-6290-4c29-a474-b6a86c1058fa"
+      (reference "C?") (unit 1) (value "100nF") (footprint "Capacitor_SMD:C_0805_2012Metric_Pad1.18x1.45mm_HandSolder")
+    )
     (path "/3d96634f-3b26-447f-8ede-f6059a78b14d"
